File: EurorackPSU.sch (KiCad schematic (older format))
At the start: 25 parts, among them J1 12V AC, J2 EURO POWER HEADER, J3 +12V, J4 0V, J5 -12V, U1 LM7812, U2 LM7912

Commit message: stripbard layout
Parts:
- removed J1: 12V AC, symbol Connector:Barrel_Jack_Switch
- removed J3: +12V, symbol Connector_Generic:Conn_01x01
- removed J4: 0V, symbol Connector_Generic:Conn_01x01
- removed J5: -12V, symbol Connector_Generic:Conn_01x01
- added J1: 12VAC, Connector_PinHeader_2.54mm:PinHeader_1x02_P2.54mm_Vertical, symbol Connector_Generic:Conn_01x02
- C1, C2, C3, C4, C5, C6: footprint (none) -> Capacitor_THT:CP_Radial_D13.0mm_P5.00mm
- C10, C7, C8, C9: footprint (none) -> Capacitor_THT:CP_Radial_Tantal_D4.5mm_P5.00mm
- D1, D2, D3, D4, D5, D6: footprint (none) -> Diode_THT:D_A-405_P7.62mm_Horizontal
- J2: footprint (none) -> Connector_PinHeader_2.54mm:PinHeader_2x05_P2.54mm_Vertical
- R1, R2: footprint (none) -> Resistor_THT:R_Axial_DIN0207_L6.3mm_D2.5mm_P7.62mm_Horizontal
Connections:
- wire segments 87 -> 81
- no-connect marks 1 -> 0
Changed lines of the file:
@@
 F 0 "C7" H 7315 4996 50  0000 L CNN
 F 1 "1uF" H 7315 4905 50  0000 L CNN
-F 2 "" H 7200 4950 50  0001 C CNN
+F 2 "Capacitor_THT:CP_Radial_Tantal_D4.5mm_P5.00mm" H 7200 4950 50  0001 C CNN
 F 3 "~" H 7200 4950 50  0001 C CNN
 	1    7200 4950
@@
 F 0 "C5" H 6815 4996 50  0000 L CNN
 F 1 "3300uF" H 6815 4905 50  0000 L CNN
-F 2 "" H 6700 4950 50  0001 C CNN
+F 2 "Capacitor_THT:CP_Radial_D13.0mm_P5.00mm" H 6700 4950 50  0001 C CNN
 F 3 "~" H 6700 4950 50  0001 C CNN
 	1    6700 4950
@@
 F 0 "R2" H 9070 4996 50  0000 L CNN
 F 1 "2.4K" H 9070 4905 50  0000 L CNN
-F 2 "" V 8930 4950 50  0001 C CNN
+F 2 "Resistor_THT:R_Axial_DIN0207_L6.3mm_D2.5mm_P7.62mm_Horizontal" V 8930 4950 50  0001 C CNN
 F 3 "~" H 9000 4950 50  0001 C CNN
 	1    9000 4950
@@
 L power:GNDD #PWR0101
 U 1 1 5B79B719
-P 5050 5850
-F 0 "#PWR0101" H 5050 5600 50  0001 C CNN
-F 1 "GNDD" H 5054 5695 50  0000 C CNN
-F 2 "" H 5050 5850 50  0001 C CNN
-F 3 "" H 5050 5850 50  0001 C CNN
-	1    5050 5850
+P 5150 5850
+F 0 "#PWR0101" H 5150 5600 50  0001 C CNN
+F 1 "GNDD" H 5154 5695 50  0000 C CNN
+F 2 "" H 5150 5850 50  0001 C CNN
+F 3 "" H 5150 5850 50  0001 C CNN
+	1    5150 5850
 	1    0    0    -1
 $EndComp
@@
 F 0 "C1" H 5815 4996 50  0000 L CNN
 F 1 "3300uF" H 5815 4905 50  0000 L CNN
-F 2 "" H 5700 4950 50  0001 C CNN
+F 2 "Capacitor_THT:CP_Radial_D13.0mm_P5.00mm" H 5700 4950 50  0001 C CNN
 F 3 "~" H 5700 4950 50  0001 C CNN
 	1    5700 4950
@@
 F 0 "C3" H 6315 4996 50  0000 L CNN
 F 1 "3300uF" H 6315 4905 50  0000 L CNN
-F 2 "" H 6200 4950 50  0001 C CNN
+F 2 "Capacitor_THT:CP_Radial_D13.0mm_P5.00mm" H 6200 4950 50  0001 C CNN
 F 3 "~" H 6200 4950 50  0001 C CNN
 	1    6200 4950
@@
 F 0 "C9" H 8215 4996 50  0000 L CNN
 F 1 "1uF" H 8215 4905 50  0000 L CNN
-F 2 "" H 8100 4950 50  0001 C CNN
+F 2 "Capacitor_THT:CP_Radial_Tantal_D4.5mm_P5.00mm" H 8100 4950 50  0001 C CNN
 F 3 "~" H 8100 4950 50  0001 C CNN
 	1    8100 4950
@@
 F 0 "D1" V 5300 4850 50  0000 C CNN
 F 1 "1N4004" V 5200 4750 50  0000 C CNN
-F 2 "" H 5250 4950 50  0001 C CNN
+F 2 "Diode_THT:D_A-405_P7.62mm_Horizontal" H 5250 4950 50  0001 C CNN
 F 3 "~" H 5250 4950 50  0001 C CNN
 	1    5250 4950
@@
 F 0 "C2" H 5585 5404 50  0000 R CNN
 F 1 "3300uF" H 5585 5495 50  0000 R CNN
-F 2 "" H 5700 5450 50  0001 C CNN
+F 2 "Capacitor_THT:CP_Radial_D13.0mm_P5.00mm" H 5700 5450 50  0001 C CNN
 F 3 "~" H 5700 5450 50  0001 C CNN
 	1    5700 5450
@@
 F 0 "C4" H 6085 5404 50  0000 R CNN
 F 1 "3300uF" H 6085 5495 50  0000 R CNN
-F 2 "" H 6200 5450 50  0001 C CNN
+F 2 "Capacitor_THT:CP_Radial_D13.0mm_P5.00mm" H 6200 5450 50  0001 C CNN
 F 3 "~" H 6200 5450 50  0001 C CNN
 	1    6200 5450
@@
 F 0 "C6" H 6585 5404 50  0000 R CNN
 F 1 "3300uF" H 6585 5495 50  0000 R CNN
-F 2 "" H 6700 5450 50  0001 C CNN
+F 2 "Capacitor_THT:CP_Radial_D13.0mm_P5.00mm" H 6700 5450 50  0001 C CNN
 F 3 "~" H 6700 5450 50  0001 C CNN
 	1    6700 5450
@@
 F 0 "C8" H 7085 5404 50  0000 R CNN
 F 1 "1uF" H 7085 5495 50  0000 R CNN
-F 2 "" H 7200 5450 50  0001 C CNN
+F 2 "Capacitor_THT:CP_Radial_Tantal_D4.5mm_P5.00mm" H 7200 5450 50  0001 C CNN
 F 3 "~" H 7200 5450 50  0001 C CNN
 	1    7200 5450
@@
 F 0 "D2" V 5300 5350 50  0000 C CNN
 F 1 "1N4004" V 5200 5250 50  0000 C CNN
-F 2 "" H 5250 5450 50  0001 C CNN
+F 2 "Diode_THT:D_A-405_P7.62mm_Horizontal" H 5250 5450 50  0001 C CNN
 F 3 "~" H 5250 5450 50  0001 C CNN
 	1    5250 5450
@@
 F 0 "D5" V 8504 5029 50  0000 L CNN
 F 1 "1N4004" V 8595 5029 50  0000 L CNN
-F 2 "" H 8550 4950 50  0001 C CNN
+F 2 "Diode_THT:D_A-405_P7.62mm_Horizontal" H 8550 4950 50  0001 C CNN
 F 3 "~" H 8550 4950 50  0001 C CNN
 	1    8550 4950
@@
 F 0 "R1" H 9070 5496 50  0000 L CNN
 F 1 "2.4K" H 9070 5405 50  0000 L CNN
-F 2 "" V 8930 5450 50  0001 C CNN
+F 2 "Resistor_THT:R_Axial_DIN0207_L6.3mm_D2.5mm_P7.62mm_Horizontal" V 8930 5450 50  0001 C CNN
 F 3 "~" H 9000 5450 50  0001 C CNN
 	1    9000 5450
@@
 F 0 "D3" H 7650 4516 50  0000 C CNN
 F 1 "1N4004" H 7650 4425 50  0000 C CNN
-F 2 "" H 7650 4300 50  0001 C CNN
+F 2 "Diode_THT:D_A-405_P7.62mm_Horizontal" H 7650 4300 50  0001 C CNN
 F 3 "~" H 7650 4300 50  0001 C CNN
 	1    7650 4300
@@
 F 0 "D4" H 7650 6316 50  0000 C CNN
 F 1 "1N4004" H 7650 6225 50  0000 C CNN
-F 2 "" H 7650 6100 50  0001 C CNN
+F 2 "Diode_THT:D_A-405_P7.62mm_Horizontal" H 7650 6100 50  0001 C CNN
 F 3 "~" H 7650 6100 50  0001 C CNN
 	1    7650 6100
@@
 F 0 "C10" H 7985 5404 50  0000 R CNN
 F 1 "1uF" H 7985 5495 50  0000 R CNN
-F 2 "" H 8100 5450 50  0001 C CNN
+F 2 "Capacitor_THT:CP_Radial_Tantal_D4.5mm_P5.00mm" H 8100 5450 50  0001 C CNN
 F 3 "~" H 8100 5450 50  0001 C CNN
 	1    8100 5450
@@
 F 0 "D6" V 8596 5371 50  0000 R CNN
 F 1 "1N4004" V 8505 5371 50  0000 R CNN
-F 2 "" H 8550 5450 50  0001 C CNN
+F 2 "Diode_THT:D_A-405_P7.62mm_Horizontal" H 8550 5450 50  0001 C CNN
 F 3 "~" H 8550 5450 50  0001 C CNN
 	1    8550 5450
@@
 	9000 4700 9000 4800
 Connection ~ 8550 4700
-$Comp
-L Connector_Generic:Conn_01x01 J3
-U 1 1 5B7D7066
-P 10300 4700
-F 0 "J3" H 10380 4742 50  0000 L CNN
-F 1 "+12V" H 10380 4651 50  0000 L CNN
-F 2 "" H 10300 4700 50  0001 C CNN
-F 3 "~" H 10300 4700 50  0001 C CNN
-	1    10300 4700
-	1    0    0    -1
-$EndComp
-$Comp
-L Connector_Generic:Conn_01x01 J4
-U 1 1 5B7D70CD
-P 10300 5200
-F 0 "J4" H 10380 5242 50  0000 L CNN
-F 1 "0V" H 10380 5151 50  0000 L CNN
-F 2 "" H 10300 5200 50  0001 C CNN
-F 3 "~" H 10300 5200 50  0001 C CNN
-	1    10300 5200
-	1    0    0    -1
-$EndComp
-$Comp
-L Connector_Generic:Conn_01x01 J5
-U 1 1 5B7D9094
-P 10300 5700
-F 0 "J5" H 10380 5742 50  0000 L CNN
-F 1 "-12V" H 10380 5651 50  0000 L CNN
-F 2 "" H 10300 5700 50  0001 C CNN
-F 3 "~" H 10300 5700 50  0001 C CNN
-	1    10300 5700
-	1    0    0    -1
-$EndComp
-$Comp
-L Connector:Barrel_Jack_Switch J1
-U 1 1 5B7D934D
-P 4500 5150
-F 0 "J1" H 4555 5467 50  0000 C CNN
-F 1 "12V AC" H 4555 5376 50  0000 C CNN
-F 2 "" H 4550 5110 50  0001 C CNN
-F 3 "~" H 4550 5110 50  0001 C CNN
-	1    4500 5150
-	1    0    0    -1
-$EndComp
 $Comp
 L Connector_Generic:Conn_02x05_Odd_Even J2
@@
 F 0 "J2" H 9800 4775 50  0000 C CNN
 F 1 "EURO POWER HEADER" H 10200 4850 50  0000 R BNN
-F 2 "" H 9750 5200 50  0001 C CNN
+F 2 "Connector_PinHeader_2.54mm:PinHeader_2x05_P2.54mm_Vertical" H 9750 5200 50  0001 C CNN
 F 3 "~" H 9750 5200 50  0001 C CNN
 	1    9750 5200
@@
 Wire Wire Line
 	9000 5200 9000 5300
-Connection ~ 9950 5700
 Wire Wire Line
 	9950 4700 9950 5000
 Wire Wire Line
 	5700 5200 6200 5200
-NoConn ~ 4800 5150
 Wire Wire Line
 	7200 5700 7350 5700
@@
 Wire Wire Line
 	9000 5700 9450 5700
-Wire Wire Line
-	9950 5700 10100 5700
-Wire Wire Line
-	9950 4700 10100 4700
 Connection ~ 9450 4700
 Wire Wire Line
 	9450 4700 9950 4700
-Connection ~ 9950 4700
 Wire Wire Line
 	9450 5700 9950 5700
@@
 Wire Wire Line
 	9000 5200 9450 5200
-Wire Wire Line
-	9950 5200 10100 5200
 Wire Wire Line
 	9450 5200 9450 5100
@@
 Wire Wire Line
 	8100 5200 8100 5100
-Wire Wire Line
-	4800 5250 5050 5250
-Wire Wire Line
-	5050 5250 5050 5200
-Wire Wire Line
-	5050 5200 5700 5200
-Wire Wire Line
-	5050 5850 5050 5250
-Connection ~ 5050 5250
-Wire Wire Line
-	4800 5050 5050 5050
-Wire Wire Line
-	5050 5050 5050 5100
-Wire Wire Line
-	5050 5100 5250 5100
 Connection ~ 5250 5100
 Wire Wire Line
 	9950 5400 9950 5700
 Connection ~ 9950 5200
+$Comp
+L Connector_Generic:Conn_01x02 J1
+U 1 1 5B829FFB
+P 4850 5100
+F 0 "J1" H 4770 5317 50  0000 C CNN
+F 1 "12VAC" H 4770 5226 50  0000 C CNN
+F 2 "Connector_PinHeader_2.54mm:PinHeader_1x02_P2.54mm_Vertical" H 4850 5100 50  0001 C CNN
+F 3 "~" H 4850 5100 50  0001 C CNN
+	1    4850 5100
+	-1   0    0    -1
+$EndComp
+Wire Wire Line
+	5150 5200 5150 5850
+Wire Wire Line
+	5050 5200 5150 5200
+Connection ~ 5150 5200
+Wire Wire Line
+	5050 5100 5250 5100
+Wire Wire Line
+	5150 5200 5700 5200
 $EndSCHEMATC
